File: HG_Con_Switch_OshPark/HG_002.kicad_pcb (KiCad board)
At the start: 2 copper layers, 87 x 94 mm, 32 parts, among them J1 CONN_01X03, J2 CONN_01X03, J3 CONN_02X03, J4 CONN_01X02, J5 CONN_01X02, U1 ATTINY85-20SU, U2 LM340MP-5.0/NOPB

Commit message: Update Back Silk
Parts:
- moved G*** 2.50 mm to (137.5, 78.9)
- moved G*** 2.06 mm to (137.5, 73.6)
- moved svg2mod 0.21 mm to (145.1, 97.4)
Other:
- board text added: "A1"
- board text added: "A3"
- board text added: "MISO"
- board text added: "MOSI"
- board text added: "RES"
- board text added: "SCK"
- board text added: "VCC"
Changed lines of the file:
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@@
-(kicad_pcb (version 20171130) (host pcbnew 6.0.0-rc1-unknown-7b10490~66~ubuntu16.04.1)
+(kicad_pcb (version 20171130) (host pcbnew 6.0.0-rc1-unknown-0bceb69~66~ubuntu16.04.1)
   (general
     (thickness 1.6)
-    (drawings 8)
+    (drawings 20)
     (tracks 238)
     (zones 0)
@@
     (35 F.Paste user)
     (36 B.SilkS user)
-    (37 F.SilkS user)
+    (37 F.SilkS user hide)
     (38 B.Mask user)
-    (39 F.Mask user)
+    (39 F.Mask user hide)
     (40 Dwgs.User user)
     (41 Cmts.User user)
@@
     (47 F.CrtYd user)
     (48 B.Fab user)
-    (49 F.Fab user hide)
+    (49 F.Fab user)
   )
   (setup
@@
     (tags "SOIC 1.27")
     (attr smd)
-    (fp_text reference U1 (at 0.1778 -3.6576 180) (layer B.SilkS)
+    (fp_text reference U1 (at 0.2286 1.6256 180) (layer B.SilkS)
       (effects (font (size 1 1) (thickness 0.15)) (justify mirror))
     )
@@
   )
   (module OshPark_Version:OSHpark-1-1100 (layer B.Cu)
-    (at 137.6172 75.692)
+    (at 137.541 73.6346)
     (fp_text reference G*** (at 0 0) (layer B.SilkS) hide
       (effects (font (size 1.524 1.524) (thickness 0.3)) (justify mirror))
@@
   )
   (module OshPark_Version:OSHpark-2-1800 (layer B.Cu)
-    (at 137.0076 81.3562 180)
+    (at 137.541 78.9178 180)
     (fp_text reference G*** (at 0 0 180) (layer B.SilkS) hide
       (effects (font (size 1.524 1.524) (thickness 0.3)) (justify mirror))
@@
   )
   (module PCBWay:HG_SilkS.Back.2 (layer B.Cu)
-    (at 145.288 97.409 180)
+    (at 145.0848 97.3582 180)
     (descr "Imported from HG_SilkS_Edge_Cuts.svg")
     (tags svg2mod)
@@
       (xy 3.606198 -46.89089) (xy 3.60606 -46.88987)) (layer F.SilkS) (width 0))
   )
+  (gr_text VCC (at 164.3126 86.6394) (layer B.SilkS)
+    (effects (font (size 1.016 1.016) (thickness 0.254)) (justify mirror))
+  )
+  (gr_text GND (at 164.1348 83.8708) (layer B.SilkS)
+    (effects (font (size 1.016 1.016) (thickness 0.254)) (justify mirror))
+  )
+  (gr_text A3 (at 164.6174 81.6102) (layer B.SilkS)
+    (effects (font (size 1.016 1.016) (thickness 0.254)) (justify mirror))
+  )
+  (gr_text A1 (at 131.953 81.5594) (layer B.SilkS)
+    (effects (font (size 1.016 1.016) (thickness 0.254)) (justify mirror))
+  )
+  (gr_text GND (at 132.6388 84.0994) (layer B.SilkS)
+    (effects (font (size 1.016 1.016) (thickness 0.254)) (justify mirror))
+  )
+  (gr_text VCC (at 132.588 86.614) (layer B.SilkS)
+    (effects (font (size 1.016 1.016) (thickness 0.254)) (justify mirror))
+  )
+  (gr_text VCC (at 146.2024 94.7166 90) (layer B.SilkS)
+    (effects (font (size 1.016 1.016) (thickness 0.254)) (justify mirror))
+  )
+  (gr_text MOSI (at 148.8186 94.9706 90) (layer B.SilkS)
+    (effects (font (size 1.016 1.016) (thickness 0.254)) (justify mirror))
+  )
+  (gr_text RES (at 151.4094 82.6262 90) (layer B.SilkS)
+    (effects (font (size 1.016 1.016) (thickness 0.254)) (justify mirror))
+  )
+  (gr_text SCK (at 148.8694 82.6008 90) (layer B.SilkS)
+    (effects (font (size 1.016 1.016) (thickness 0.254)) (justify mirror))
+  )
+  (gr_text GND (at 151.4602 94.7166 90) (layer B.SilkS)
+    (effects (font (size 1.016 1.016) (thickness 0.254)) (justify mirror))
+  )
+  (gr_text MISO (at 146.2278 82.3214 90) (layer B.SilkS)
+    (effects (font (size 1.016 1.016) (thickness 0.254)) (justify mirror))
+  )
   (gr_text VIN (at 130.7338 99.2378) (layer B.SilkS)
     (effects (font (size 1.5 1.5) (thickness 0.3)) (justify mirror))
@@
     (connect_pads (clearance 0.508))
     (min_thickness 0.254)
-    (fill yes (arc_segments 16) (thermal_gap 0.508) (thermal_bridge_width 0.508))
+    (fill (arc_segments 16) (thermal_gap 0.508) (thermal_bridge_width 0.508))
     (polygon
       (pts
@@
     (connect_pads (clearance 0.508))
     (min_thickness 0.254)
-    (fill yes (arc_segments 16) (thermal_gap 0.508) (thermal_bridge_width 0.508))
+    (fill (arc_segments 16) (thermal_gap 0.508) (thermal_bridge_width 0.508))
     (polygon
       (pts
