File: HG_Con_Switch_OshPark/HG_002.sch (KiCad schematic (older format))
At the start: 25 parts, among them J1 CONN_01X03, J2 CONN_01X03, J3 CONN_02X03, J4 CONN_01X02, J5 CONN_01X02, U1 ATTINY85-20SU, U2 LM340MP-5.0/NOPB

Commit message: Update Back Silk
Parts:
- D1: symbol 001-rescue:LED-RESCUE-001 -> HG_002-rescue:LED-RESCUE-001-001-rescue
Changed lines of the file:
@@
 $EndComp
 $Comp
-L 001-rescue:LED-RESCUE-001 D1
+L HG_002-rescue:LED-RESCUE-001-001-rescue D1
 U 1 1 597EC09A
 P 2315 7385
